Commit message: Added limits

File: Code/App/scripts/assets/URDF/armURDF.URDF (robot description, URDF)
Before this commit: robot JN_V1, 9 links, 8 joints
Joints:
- joint elbow_rot: limit (none) -> lower=-2.622 upper=0
- joint shoulder_rot: limit (none) -> lower=0 upper=3.14
- joint wrist_rot: limit (none) -> lower=-1.57 upper=1.57

Commit message: Added a smaller upper limit since the limit switch blocks the motor from reaching 3.14 anyways

File: Code/App/scripts/assets/URDF/armURDF.URDF (robot description, URDF)
Before this commit: robot JN_V1, 9 links, 8 joints
Joints:
- joint shoulder_rot: limit lower=0 upper=3.14 -> lower=0 upper=2.35619

Commit message: Made the limit more accurate to real life

File: Code/App/scripts/assets/URDF/armURDF.URDF (robot description, URDF)
Before this commit: robot JN_V1, 9 links, 8 joints
Joints:
- joint wrist_rot: limit lower=-1.57 upper=1.57 -> lower=-1.39626 upper=1.57
